Commit message: added wheels

File: urdf/udacity_bot.xacro (robot description, xacro)
@@ -75,3 +75,65 @@
     </visual>
   </link>
+  <link name="left_wheel">
+    <inertial>
+      <mass value="5.0"/>
+      <origin xyz="0.0 0 0" rpy=" 0 0 0"/>
+      <inertia
+          ixx="0.1" ixy="0" ixz="0"
+          iyy="0.1" iyz="0"
+          izz="0.1"
+      />
+    </inertial>
+    <collision>
+      <origin xyz="0 0 0" rpy="1.5707 0 0"/>
+      <geometry>
+        <cylinder radius=".1" length="0.05"/>
+      </geometry>
+    </collision>
+    <visual>
+      <origin xyz="0 0 0" rpy="1.5707 0 0"/>
+      <geometry>
+        <cylinder radius="0.1" length="0.05"/>
+      </geometry>
+    </visual>
+  </link>
+  <joint name="left_wheel_hinge" type="continuous">
+    <origin xyz="0.0 0.13 0" rpy="0 0 0"/>
+    <child link="left_wheel"/>
+    <parent link="chassis" />
+    <axis xyz="0 1 0" rpy="0 0 0" />
+    <limit effort="10000" velocity="1000" />
+    <joint_properties damping="1.0" friction="1.0" />
+  </joint>
+  <link name="right_wheel">
+    <inertial>
+      <mass value="5.0"/>
+      <origin xyz="0.0 0 0" rpy=" 0 0 0"/>
+      <inertia
+          ixx="0.1" ixy="0" ixz="0"
+          iyy="0.1" iyz="0"
+          izz="0.1"
+      />
+    </inertial>
+    <collision>
+      <origin xyz="0 0 0" rpy="1.5707 0 0"/>
+      <geometry>
+        <cylinder radius=".1" length="0.05"/>
+      </geometry>
+    </collision>
+    <visual>
+      <origin xyz="0 0 0" rpy="1.5707 0 0"/>
+      <geometry>
+        <cylinder radius="0.1" length="0.05"/>
+      </geometry>
+    </visual>
+  </link>
+  <joint name="right_wheel_hinge" type="continuous">
+    <origin xyz="0.0 -0.13 0" rpy="0 0 0"/>
+    <child link="right_wheel"/>
+    <parent link="chassis" />
+    <axis xyz="0 1 0" rpy="0 0 0" />
+    <limit effort="10000" velocity="1000" />
+    <joint_properties damping="1.0" friction="1.0" />
+  </joint>
 </robot>

Commit message: added camera

File: urdf/udacity_bot.xacro (robot description, xacro)
@@ -137,3 +137,31 @@
     <joint_properties damping="1.0" friction="1.0" />
   </joint>
+  <joint name="camera_joint" type="fixed">
+    <origin xyz="0.2 0 0" rpy="0 0 0" />
+    <child link="camera" />
+    <parent link="chassis" />
+  </joint>
+  <link name="camera">
+    <inertial>
+      <mass value="0.1"/>
+      <origin xyz="0.0 0 0" rpy=" 0 0 0"/>
+      <inertia
+          ixx="1e-6" ixy="0" ixz="0"
+          iyy="1e-6" iyz="0"
+          izz="1e-6"
+      />
+    </inertial>
+    <collision>
+      <origin xyz="0 0 0" rpy=" 0 0 0"/>
+      <geometry>
+        <box size="0.05 0.05 0.05" />
+      </geometry>
+    </collision>
+    <visual>
+      <origin xyz="0 0 0" rpy=" 0 0 0"/>
+      <geometry>
+        <box size="0.05 0.05 0.05" />
+      </geometry>
+    </visual>
+  </link>
 </robot>

Commit message: added laser finder

File: urdf/udacity_bot.xacro (robot description, xacro)
@@ -75,4 +75,35 @@
     </visual>
   </link>
+  <link name="right_wheel">
+    <inertial>
+      <mass value="5.0"/>
+      <origin xyz="0.0 0 0" rpy=" 0 0 0"/>
+      <inertia
+          ixx="0.1" ixy="0" ixz="0"
+          iyy="0.1" iyz="0"
+          izz="0.1"
+      />
+    </inertial>
+    <collision>
+      <origin xyz="0 0 0" rpy="1.5707 0 0"/>
+      <geometry>
+        <cylinder radius=".1" length="0.05"/>
+      </geometry>
+    </collision>
+    <visual>
+      <origin xyz="0 0 0" rpy="1.5707 0 0"/>
+      <geometry>
+        <cylinder radius="0.1" length="0.05"/>
+      </geometry>
+    </visual>
+  </link>
+  <joint name="right_wheel_hinge" type="continuous">
+    <origin xyz="0.0 -0.13 0" rpy="0 0 0"/>
+    <child link="right_wheel"/>
+    <parent link="chassis" />
+    <axis xyz="0 1 0" rpy="0 0 0" />
+    <limit effort="10000" velocity="1000" />
+    <joint_properties damping="1.0" friction="1.0" />
+  </joint>
   <link name="left_wheel">
     <inertial>
@@ -101,35 +132,4 @@
     <origin xyz="0.0 0.13 0" rpy="0 0 0"/>
     <child link="left_wheel"/>
-    <parent link="chassis" />
-    <axis xyz="0 1 0" rpy="0 0 0" />
-    <limit effort="10000" velocity="1000" />
-    <joint_properties damping="1.0" friction="1.0" />
-  </joint>
-  <link name="right_wheel">
-    <inertial>
-      <mass value="5.0"/>
-      <origin xyz="0.0 0 0" rpy=" 0 0 0"/>
-      <inertia
-          ixx="0.1" ixy="0" ixz="0"
-          iyy="0.1" iyz="0"
-          izz="0.1"
-      />
-    </inertial>
-    <collision>
-      <origin xyz="0 0 0" rpy="1.5707 0 0"/>
-      <geometry>
-        <cylinder radius=".1" length="0.05"/>
-      </geometry>
-    </collision>
-    <visual>
-      <origin xyz="0 0 0" rpy="1.5707 0 0"/>
-      <geometry>
-        <cylinder radius="0.1" length="0.05"/>
-      </geometry>
-    </visual>
-  </link>
-  <joint name="right_wheel_hinge" type="continuous">
-    <origin xyz="0.0 -0.13 0" rpy="0 0 0"/>
-    <child link="right_wheel"/>
     <parent link="chassis" />
     <axis xyz="0 1 0" rpy="0 0 0" />
@@ -165,3 +165,32 @@
     </visual>
   </link>
+  <link name='hokuyo'>
+    <inertial>
+      <mass value="0.1"/>
+      <origin xyz="0 0 0" rpy="0 0 0"/>
+      <inertia
+          ixx="1e-6" ixy="0" ixz="0"
+          iyy="1e-6" iyz="0"
+          izz="1e-6"
+      />
+    </inertial>
+    <collision>
+      <origin xyz="0 0 0" rpy="0 0 0"/>
+      <geometry>
+        <box size=".1 .1 .1"/>
+      </geometry>
+    </collision>
+    <visual>
+      <origin xyz="0 0 0" rpy="0 0 0"/>
+      <geometry>
+        <mesh filename="package://udacity_bot/meshes/hokuyo.dae"/>
+      </geometry>
+    </visual>
+  </link>
+  <joint type="fixed" name="hokuyo_joint">
+    <origin xyz="0.15 0 0.08" rpy="0 0 0"/>
+    <child link="hokuyo"/>
+    <parent link="chassis"/>
+    <axis xyz="0 1 0" rpy="0 0 0"/>
+  </joint>
 </robot>

Commit message: updated amcl launch

File: urdf/udacity_bot.xacro (robot description, xacro)
@@ -76,8 +76,8 @@
     </visual>
   </link>
-  <link name="right_wheel">
+  <link name='left_wheel'>
     <inertial>
       <mass value="5.0"/>
-      <origin xyz="0.0 0 0" rpy=" 0 0 0"/>
+      <origin xyz="0 0 0" rpy="0 1.57 1.57"/>
       <inertia
           ixx="0.1" ixy="0" ixz="0"
@@ -87,28 +87,20 @@
     </inertial>
     <collision>
-      <origin xyz="0 0 0" rpy="1.5707 0 0"/>
+      <origin xyz="0 0 0" rpy="0 1.57 1.57"/>
       <geometry>
-        <cylinder radius=".1" length="0.05"/>
+        <cylinder length="0.05" radius="0.1"/>
       </geometry>
     </collision>
     <visual>
-      <origin xyz="0 0 0" rpy="1.5707 0 0"/>
+      <origin xyz="0 0 0" rpy="0 1.57 1.57"/>
       <geometry>
-        <cylinder radius="0.1" length="0.05"/>
+        <cylinder length="0.05" radius="0.1"/>
       </geometry>
     </visual>
   </link>
-  <joint name="right_wheel_hinge" type="continuous">
-    <origin xyz="0.0 -0.13 0" rpy="0 0 0"/>
-    <child link="right_wheel"/>
-    <parent link="chassis" />
-    <axis xyz="0 1 0" rpy="0 0 0" />
-    <limit effort="10000" velocity="1000" />
-    <joint_properties damping="1.0" friction="1.0" />
-  </joint>
-  <link name="left_wheel">
+  <link name='right_wheel'>
     <inertial>
       <mass value="5.0"/>
-      <origin xyz="0.0 0 0" rpy=" 0 0 0"/>
+      <origin xyz="0 0 0" rpy="0 1.57 1.57"/>
       <inertia
           ixx="0.1" ixy="0" ixz="0"
@@ -118,33 +110,36 @@
     </inertial>
     <collision>
-      <origin xyz="0 0 0" rpy="1.5707 0 0"/>
+      <origin xyz="0 0 0" rpy="0 1.57 1.57"/>
       <geometry>
-        <cylinder radius=".1" length="0.05"/>
+        <cylinder length="0.05" radius="0.1"/>
       </geometry>
     </collision>
     <visual>
-      <origin xyz="0 0 0" rpy="1.5707 0 0"/>
+      <origin xyz="0 0 0" rpy="0 1.57 1.57"/>
       <geometry>
-        <cylinder radius="0.1" length="0.05"/>
+        <cylinder length="0.05" radius="0.1"/>
       </geometry>
     </visual>
   </link>
-  <joint name="left_wheel_hinge" type="continuous">
-    <origin xyz="0.0 0.13 0" rpy="0 0 0"/>
+  <joint type="continuous" name="left_wheel_hinge">
+    <origin xyz="0 0.15 0" rpy="0 0 0"/>
     <child link="left_wheel"/>
-    <parent link="chassis" />
-    <axis xyz="0 1 0" rpy="0 0 0" />
-    <limit effort="10000" velocity="1000" />
-    <joint_properties damping="1.0" friction="1.0" />
+    <parent link="chassis"/>
+    <axis xyz="0 1 0" rpy="0 0 0"/>
+    <limit effort="10000" velocity="1000"/>
+    <joint_properties damping="1.0" friction="1.0"/>
   </joint>
-  <joint name="camera_joint" type="fixed">
-    <origin xyz="0.2 0 0" rpy="0 0 0" />
-    <child link="camera" />
-    <parent link="chassis" />
+  <joint type="continuous" name="right_wheel_hinge">
+    <origin xyz="0 -0.15 0" rpy="0 0 0"/>
+    <child link="right_wheel"/>
+    <parent link="chassis"/>
+    <axis xyz="0 1 0" rpy="0 0 0"/>
+    <limit effort="10000" velocity="1000"/>
+    <joint_properties damping="1.0" friction="1.0"/>
   </joint>
-  <link name="camera">
+  <link name='camera'>
     <inertial>
       <mass value="0.1"/>
-      <origin xyz="0.0 0 0" rpy=" 0 0 0"/>
+      <origin xyz="0 0 0" rpy="0 0 0"/>
       <inertia
           ixx="1e-6" ixy="0" ixz="0"
@@ -154,16 +149,22 @@
     </inertial>
     <collision>
-      <origin xyz="0 0 0" rpy=" 0 0 0"/>
+      <origin xyz="0 0 0" rpy="0 0 0"/>
       <geometry>
-        <box size="0.05 0.05 0.05" />
+        <box size=".05 .05 .05"/>
       </geometry>
     </collision>
     <visual>
-      <origin xyz="0 0 0" rpy=" 0 0 0"/>
+      <origin xyz="0 0 0" rpy="0 0 0"/>
       <geometry>
-        <box size="0.05 0.05 0.05" />
+        <box size=".05 .05 .05"/>
       </geometry>
     </visual>
   </link>
+  <joint type="fixed" name="camera_joint">
+    <origin xyz="0.2 0 0" rpy="0 0 0"/>
+    <child link="camera"/>
+    <parent link="chassis"/>
+    <axis xyz="0 1 0" rpy="0 0 0"/>
+  </joint>
   <link name='hokuyo'>
     <inertial>
@@ -190,5 +191,5 @@
   </link>
   <joint type="fixed" name="hokuyo_joint">
-    <origin xyz="0.15 0 0.08" rpy="0 0 0"/>
+    <origin xyz="0.15 0 0.1" rpy="0 0 0"/>
     <child link="hokuyo"/>
     <parent link="chassis"/>

Commit message: amcl and urdf

File: urdf/udacity_bot.xacro (robot description, xacro)
@@ -2,4 +2,10 @@
 <robot name="udacity_bot" xmlns:xacro="http://www.ros.org/wiki/xacro">
   <xacro:include filename="$(find udacity_bot)/urdf/udacity_bot.gazebo" />
+  <material name="blue">
+     <color rgba="0 0 0.8 1"/>
+  </material>
+  <material name="green">
+     <color rgba="0 .8 0 1"/>
+  </material>
   <link name="robot_footprint"></link>
   <joint name="robot_footprint_joint" type="fixed">
@@ -26,4 +32,5 @@
     </collision>
     <visual name='chassis_visual'>
+    <material name="blue"/>
       <origin xyz="0 0 0" rpy=" 0 0 0"/>
       <geometry>
@@ -76,5 +83,5 @@
     </visual>
   </link>
-  <link name='left_wheel'>
+  <link name='right_wheel'>
     <inertial>
       <mass value="5.0"/>
@@ -94,10 +101,11 @@
     <visual>
       <origin xyz="0 0 0" rpy="0 1.57 1.57"/>
-      <geometry>
-        <cylinder length="0.05" radius="0.1"/>
-      </geometry>
-    </visual>
-  </link>
-  <link name='right_wheel'>
+      <material name="green"/>
+      <geometry>
+        <cylinder length="0.05" radius="0.1"/>
+      </geometry>
+    </visual>
+  </link>
+  <link name='left_wheel'>
     <inertial>
       <mass value="5.0"/>
@@ -117,9 +125,18 @@
     <visual>
       <origin xyz="0 0 0" rpy="0 1.57 1.57"/>
-      <geometry>
-        <cylinder length="0.05" radius="0.1"/>
-      </geometry>
-    </visual>
-  </link>
+      <material name="green"/>
+      <geometry>
+        <cylinder length="0.05" radius="0.1"/>
+      </geometry>
+    </visual>
+  </link>
+  <joint type="continuous" name="right_wheel_hinge">
+    <origin xyz="0 -0.15 0" rpy="0 0 0"/>
+    <child link="right_wheel"/>
+    <parent link="chassis"/>
+    <axis xyz="0 1 0" rpy="0 0 0"/>
+    <limit effort="10000" velocity="1000"/>
+    <joint_properties damping="1.0" friction="1.0"/>
+  </joint>
   <joint type="continuous" name="left_wheel_hinge">
     <origin xyz="0 0.15 0" rpy="0 0 0"/>
@@ -130,12 +147,4 @@
     <joint_properties damping="1.0" friction="1.0"/>
   </joint>
-  <joint type="continuous" name="right_wheel_hinge">
-    <origin xyz="0 -0.15 0" rpy="0 0 0"/>
-    <child link="right_wheel"/>
-    <parent link="chassis"/>
-    <axis xyz="0 1 0" rpy="0 0 0"/>
-    <limit effort="10000" velocity="1000"/>
-    <joint_properties damping="1.0" friction="1.0"/>
-  </joint>
   <link name='camera'>
     <inertial>

Commit message: rviz green camera

File: urdf/udacity_bot.xacro (robot description, xacro)
@@ -165,4 +165,5 @@
     <visual>
       <origin xyz="0 0 0" rpy="0 0 0"/>
+      <material name="green"/>
       <geometry>
         <box size=".05 .05 .05"/>
